Commit message: Added second table

File: cylinder.urdf (robot description, URDF)
Before this commit: robot cylinder, 1 links, 0 joints
Links:
- link base_link: geometry collision cylinder length=0.02 radius=0.08; visual cylinder length=0.02 radius=0.08

Commit message: Clean repo and added readme and requirements

File: cylinder.urdf (robot description, URDF)
Before this commit: robot cylinder, 1 links, 0 joints
Links:
- link base_link: mass 0.5 -> 50; geometry collision cylinder length=0.4 radius=0.1; visual cylinder length=0.02 radius=0.08
